File: Boards/Flamingo PCBA/Flamingo PCB Rev 1/Flamingo PCB Rev 1.1/Flamingo PCB Rev 1.1.brd (EAGLE design)
At the start: 100 x 80 mm, 11 parts

Commit message: Completed preliminary component layout
Decided to just glue the 5 wires from the remote and 4 for the lights
to the underside of the PCB.
Parts:
- removed JP1, JP2: (no value), adafruit:1X12-CB
- removed JP3: (no value), adafruit:1X06-CLEANBIG
- removed JP5: (no value), adafruit:1X03-CLEANBIG
- added J2: (no value), SparkFun-Connectors:1X05
- added J3: (no value), SparkFun-Connectors:1X02
- R1, R2: value (none) -> 2K2
- moved J1 245.8 mm to (40.6, 31.8)
- moved R2 231.1 mm to (44.5, 35.6)
- moved R1 215.3 mm to (44.5, 38.1)
- moved JP4 136.3 mm to (49.5, 29.2), turned to 180 degrees
- moved U$1 134.4 mm to (48.3, 49.1)
- moved C1 117.4 mm to (55.9, 36.8), turned to 90 degrees
Connections:
- new net BTN1BRIGHT: J2.4, R1.P$2, U$1.3
- new net BTN2PROG: J2.3, R2.P$2, U$1.4
- new net CLK_LIGHT: J1.2, U$1.13
- new net MOSI_LIGHT: J1.3, U$1.11
- new net SCL_ACC: JP4.1, U$1.A5
- new net SDA_ACC: JP4.2, U$1.A4
- new net SWITCHA: J2.1, J3.2
- new net SWITCHB: J2.2, J3.1
- net BAT+: now also C1.+, J1.4, JP4.6, JP4.7
- net GND: now also C1.-, J1.1, J2.5, JP4.3, JP4.8, R1.P$1, R2.P$1
Routing:
- added copper zone on layer 1, net N$1
Other:
- board text added: "Paul Blackburn"
Changed lines of the file:
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@@
 <setting verticaltext="up"/>
 </settings>
-<grid distance="50" unitdist="mil" unit="mil" style="lines" multiple="1" display="no" altdistance="5" altunitdist="mil" altunit="mil"/>
+<grid distance="50" unitdist="mil" unit="mil" style="lines" multiple="1" display="yes" altdistance="5" altunitdist="mil" altunit="mil"/>
 <layers>
 <layer number="1" name="Top" color="4" fill="1" visible="yes" active="yes"/>
@@
 <wire x1="100" y1="80" x2="0" y2="80" width="0" layer="20"/>
 <wire x1="0" y1="80" x2="0" y2="0" width="0" layer="20"/>
+<text x="53.34" y="-7.62" size="1.778" layer="1">Paul Blackburn</text>
 </plain>
 <attributes>
@@
 <elements>
 <element name="FRAME1" library="SparkFun-Aesthetics" library_urn="urn:adsk.eagle:library:507" package="CREATIVE_COMMONS" value="FRAME-LETTER" x="21.59" y="-7.62"/>
-<element name="JP1" library="adafruit" library_urn="urn:adsk.eagle:library:420" package="1X12-CB" value="" x="22.86" y="-17.78"/>
-<element name="JP2" library="adafruit" library_urn="urn:adsk.eagle:library:420" package="1X12-CB" value="" x="22.86" y="-35.56"/>
-<element name="JP3" library="adafruit" library_urn="urn:adsk.eagle:library:420" package="1X06-CLEANBIG" value="" x="15.24" y="-53.34"/>
-<element name="C1" library="adafruit" library_urn="urn:adsk.eagle:library:420" package="E5-6" value="" x="12.7" y="-72.39"/>
-<element name="U$1" library="adafruit" library_urn="urn:adsk.eagle:library:420" package="PROTRINKET" value="PRO_TRINKET" x="-16.51" y="-68.58"/>
-<element name="JP4" library="adafruit" library_urn="urn:adsk.eagle:library:420" package="1X08-CLEANBIG" value="" x="-13.97" y="-91.44"/>
-<element name="JP5" library="adafruit" library_urn="urn:adsk.eagle:library:420" package="1X03-CLEANBIG" value="" x="-20.32" y="-149.86"/>
-<element name="R1" library="SparkFun-Resistors" library_urn="urn:adsk.eagle:library:532" package="AXIAL-0.3" value=" " x="-19.05" y="-167.64">
-<attribute name="PROD_ID" value=" " x="-19.05" y="-167.64" size="1.778" layer="27" display="off"/>
+<element name="C1" library="adafruit" library_urn="urn:adsk.eagle:library:420" package="E5-6" value="" x="55.88" y="36.83" rot="R90"/>
+<element name="JP4" library="adafruit" library_urn="urn:adsk.eagle:library:420" package="1X08-CLEANBIG" value="" x="49.53" y="29.21" rot="R180"/>
+<element name="R1" library="SparkFun-Resistors" library_urn="urn:adsk.eagle:library:532" package="AXIAL-0.3" value="2K2" x="44.45" y="38.1">
+<attribute name="PROD_ID" value=" " x="44.45" y="38.1" size="1.778" layer="27" display="off"/>
 </element>
-<element name="R2" library="SparkFun-Resistors" library_urn="urn:adsk.eagle:library:532" package="AXIAL-0.3" value=" " x="-19.05" y="-186.69">
-<attribute name="PROD_ID" value=" " x="-19.05" y="-186.69" size="1.778" layer="27" display="off"/>
+<element name="R2" library="SparkFun-Resistors" library_urn="urn:adsk.eagle:library:532" package="AXIAL-0.3" value="2K2" x="44.45" y="35.56">
+<attribute name="PROD_ID" value=" " x="44.45" y="35.56" size="1.778" layer="27" display="off"/>
 </element>
-<element name="J1" library="SparkFun-Connectors" library_urn="urn:adsk.eagle:library:513" package="1X04" value="" x="-22.86" y="-205.74">
-<attribute name="PROD_ID" value="CONN-09696" x="-22.86" y="-205.74" size="1.778" layer="27" display="off"/>
+<element name="J1" library="SparkFun-Connectors" library_urn="urn:adsk.eagle:library:513" package="1X04" value="" x="40.64" y="31.75">
+<attribute name="PROD_ID" value="CONN-09696" x="40.64" y="31.75" size="1.778" layer="27" display="off"/>
 </element>
+<element name="U$1" library="adafruit" library_urn="urn:adsk.eagle:library:420" package="PROTRINKET" value="PRO_TRINKET" x="48.26" y="49.149"/>
+<element name="J2" library="SparkFun-Connectors" library_urn="urn:adsk.eagle:library:513" package="1X05" value="" x="58.42" y="58.42" rot="R270"/>
+<element name="J3" library="SparkFun-Connectors" library_urn="urn:adsk.eagle:library:513" package="1X02" value="" x="58.42" y="66.04" rot="R270"/>
 </elements>
 <signals>
+<signal name="GND">
+<contactref element="JP4" pad="8"/>
+<contactref element="J1" pad="1"/>
+<contactref element="R1" pad="P$1"/>
+<contactref element="R2" pad="P$1"/>
+<contactref element="JP4" pad="3"/>
+<contactref element="C1" pad="-"/>
+<contactref element="U$1" pad="GND"/>
+<contactref element="J2" pad="5"/>
+<wire x1="40.64" y1="31.75" x2="55.88" y2="69.85" width="0" layer="19" extent="1-1"/>
+<wire x1="40.64" y1="35.56" x2="40.64" y2="31.75" width="0" layer="19" extent="1-1"/>
+<wire x1="40.64" y1="38.1" x2="40.64" y2="35.56" width="0" layer="19" extent="1-1"/>
+<wire x1="53.34" y1="29.21" x2="40.64" y2="38.1" width="0" layer="19" extent="1-1"/>
+<wire x1="40.64" y1="29.21" x2="40.64" y2="38.1" width="0" layer="19" extent="1-1"/>
+<wire x1="55.88" y1="39.37" x2="53.34" y2="29.21" width="0" layer="19" extent="1-1"/>
+<wire x1="58.42" y1="48.26" x2="40.64" y2="29.21" width="0" layer="19" extent="1-1"/>
+</signal>
+<signal name="BTN2PROG">
+<contactref element="R2" pad="P$2"/>
+<contactref element="U$1" pad="4"/>
+<contactref element="J2" pad="3"/>
+<wire x1="48.26" y1="35.56" x2="55.88" y2="54.61" width="0" layer="19" extent="1-1"/>
+<wire x1="58.42" y1="53.34" x2="48.26" y2="35.56" width="0" layer="19" extent="1-1"/>
+</signal>
+<signal name="BTN1BRIGHT">
+<contactref element="R1" pad="P$2"/>
+<contactref element="U$1" pad="3"/>
+<contactref element="J2" pad="4"/>
+<wire x1="48.26" y1="38.1" x2="55.88" y2="52.07" width="0" layer="19" extent="1-1"/>
+<wire x1="58.42" y1="50.8" x2="48.26" y2="38.1" width="0" layer="19" extent="1-1"/>
+</signal>
+<signal name="CLK_LIGHT">
+<contactref element="J1" pad="2"/>
+<contactref element="U$1" pad="13"/>
+<wire x1="40.64" y1="62.23" x2="43.18" y2="31.75" width="0" layer="19" extent="1-1"/>
+</signal>
+<signal name="SDA_ACC">
+<contactref element="JP4" pad="2"/>
+<contactref element="U$1" pad="A4"/>
+<wire x1="40.64" y1="46.99" x2="55.88" y2="29.21" width="0" layer="19" extent="1-1"/>
+</signal>
+<signal name="SCL_ACC">
+<contactref element="JP4" pad="1"/>
+<contactref element="U$1" pad="A5"/>
+<wire x1="40.64" y1="44.45" x2="58.42" y2="29.21" width="0" layer="19" extent="1-1"/>
+</signal>
+<signal name="MOSI_LIGHT">
+<contactref element="J1" pad="3"/>
+<contactref element="U$1" pad="11"/>
+<wire x1="40.64" y1="67.31" x2="45.72" y2="31.75" width="0" layer="19" extent="1-1"/>
+</signal>
 <signal name="BAT+">
 <contactref element="U$1" pad="BAT+"/>
-</signal>
-<signal name="GND">
-<contactref element="U$1" pad="GND"/>
+<contactref element="JP4" pad="7"/>
+<contactref element="JP4" pad="6"/>
+<contactref element="J1" pad="4"/>
+<contactref element="C1" pad="+"/>
+<wire x1="48.26" y1="31.75" x2="55.88" y2="34.29" width="0" layer="19" extent="1-1"/>
+<wire x1="43.18" y1="29.21" x2="48.26" y2="31.75" width="0" layer="19" extent="1-1"/>
+<wire x1="45.72" y1="29.21" x2="43.18" y2="29.21" width="0" layer="19" extent="1-1"/>
+<wire x1="55.88" y1="72.39" x2="48.26" y2="31.75" width="0" layer="19" extent="1-1"/>
 </signal>
 <signal name="USB">
@@
 <contactref element="U$1" pad="VCC"/>
 </signal>
+<signal name="SWITCHB">
+<contactref element="J3" pad="1"/>
+<contactref element="J2" pad="2"/>
+<wire x1="58.42" y1="55.88" x2="58.42" y2="66.04" width="0" layer="19" extent="1-1"/>
+</signal>
+<signal name="SWITCHA">
+<contactref element="J3" pad="2"/>
+<contactref element="J2" pad="1"/>
+<wire x1="58.42" y1="58.42" x2="58.42" y2="63.5" width="0" layer="19" extent="1-1"/>
+</signal>
+<signal name="N$1">
+<polygon width="0.1524" layer="1">
+<vertex x="39.37" y="29.21"/>
+<vertex x="59.69" y="29.21"/>
+<vertex x="59.69" y="21.59"/>
+<vertex x="39.37" y="21.59"/>
+</polygon>
+</signal>
 </signals>
