File: Boards/Flamingo PCBA/Flamingo PCB Rev 2/Flamingo_PCBaaa.sch (KiCad schematic (older format))
At the start: 11 parts

Commit message: PCB: bringing in symbols, re-making battery charger sheet, still has todo
Parts:
- J?: symbol MyConnectors:01x02_Connector -> Flamingo_PCB-rescue:Conn_01x02
Changed lines of the file:
@@
 $EndComp
 $Comp
-L MyConnectors:01x02_Connector J?
+L Flamingo_PCB-rescue:Conn_01x02 J?
 U 1 1 5A77CDB7
 P 5450 4400
