File: Boards/Flamingo PCBA/Flamingo PCB Rev 3/Flamingo PCB/Flamingo PCB - Battery Charger.sch (KiCad schematic (older format))
At the start: 0 parts

Commit message: PCB: bringing in symbols, re-making battery charger sheet, still has todo
Parts:
- added C? (x2): 10uF, symbol Device:CP1_Small
- added D?: Green/Done, symbol MyLEDs:LED_ALT_vert
- added D?: Red/Charging, symbol MyLEDs:LED_ALT_vert
- added J?: JST Battery conn, symbol MyConnectors:01x02_Connector
- added J?: Wire Switch Here, symbol MyConnectors:01x02_Connector
- added R? (x3): 2.0k, symbol MyResistors:R_vert
- added U?: MCP73831T-2ATI_OT, digikey-footprints:SOT-753, symbol dk_PMIC-Battery-Chargers:MCP73831T-2ATI_OT
Connections:
- net labels added: GND, V_BAT, V_BUS
- wire segments 0 -> 25
Other:
- note added: "--------FLOW CHART--------\n\n###SHUTDOWN MODE\nVDD < VUVLO\nVDD < VBAT\nor\nPROG > 200 k\nSTAT = High Z\n\n###PRECONDITIONING \nCharge Current = IPREG\nSTAT = LOW\n\n###FAST CHARGE \nAlso get here if VBAT > VPTH from SHUTDOWN \nor \nVBAT < VRTH from CHARGE COMPLETE\n\nCharge Current = IREG\nSTAT = LOW\n\n###CONSTANT VOLTAGE \nCharge Voltage = VREG\nSTAT = LOW\n\n###CHARGE MODE \nSTAT = HIGH (MCP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"
- note added: "Batt charging rate:\n10k = 100mA\n5.0k = 200 mA\n2.0k = 500 mA\n1.0k = 1000mA"
- note added: "TODO\nChange resistor values\nFind green resistor"
