File: Boards/Flamingo PCBA/Flamingo PCB Rev 3/Flamingo PCB/Flamingo PCB - Power.sch (KiCad schematic (older format))
At the start: 0 parts

Commit message: Worked on Power board mainly.
Still have to resolve the power sharing.
Parts:
- added C? (x6): 10uF, symbol MyCapacitors:C_Small_vert
- added D? (x6): Schottky, digikey-footprints:SOD-123, symbol dk_Diodes-Rectifiers-Single:1N5819HW-7-F
- added U?: 3.3V_Reg, digikey-footprints:SOT-753, symbol MyICs:3.3V_Reg
- added U?: 5V_Reg, digikey-footprints:SOT-753, symbol MyICs:3.3V_Reg
- added U?: 1.8V_Reg, digikey-footprints:SOT-753, symbol MyICs:3.3V_Reg
Connections:
- new net: C?.1, D?.K, D?.K, U?.1 (VIN), U?.3 (ON/~OFF) (x2)
- new net: D?.A, U?.5 (VOUT)
- new net +1.8V: C?.1, U?.5 (VOUT)
- new net +3.3V: C?.1, U?.5 (VOUT)
- new net +5V: C?.1, D?.K, D?.K
- new net GND: C?.2, C?.2, C?.2, C?.2, C?.2, C?.2, U?.2 (GND), U?.2 (GND), U?.2 (GND)
- new net V_BAT: C?.1, D?.A, D?.A, U?.1 (VIN), U?.3 (ON/~OFF)
- new net V_BUS: D?.A, D?.A, D?.A
- no-connect marks 0 -> 3
Other:
- note added: "Cases:\nCasesI would like to protect for:\n\nV_BAT open\nV_BAT shorted to ground\nV_BAT below any of 1.8V, 3.3V, 5V\nV_BAT above any of 1.8V, 3.3V up to 4.20 V\nV_BAT reversed?\n\nV_BUS 0V\nV_BUS shorted to ground"
- note added: "LP2985\n\nVin Max: 16 V\n\n--\n\n\nA minimum value of 1 μF (over the entire operating temperature range)\n is required at the input of the LP2985. In addition, this input capacitor \nshould be located within 1 cm of the input pin and connected to a\n clean analog ground. There are no equivalent series resistance (ESR) \nrequirements for this capacitor, and the capacitance can be increased without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"
- note added: "V_BAT will always be below V_BUS. If I connect Schottky diode\n from output to input as directed, now have V_BUS on the V_BAT line,\n which would bypass the battery controller. Not good.\n\nInstead maybe I can put a Schottky on the output\n so the internal diode cannot forward bias."
- note added: "V_BUS comes from USB/FTDI exclusively\n\nIf V_BUS is energized, then V_BAT is energized through battery charger.\nHowever V_BAT may be accidental short to ground, low (on battery), etc.\n\nWe want to drive the voltage regulators from V_BUS over V_BAT if available.\n\nOn/Off switch controls V_BAT, so if V_BUS is powered, switch does nothing."
