File: Boards/Flamingo PCBA/Flamingo PCB Rev 3/Flamingo PCB/Flamingo PCB - Power.sch (KiCad schematic (older format))
At the start: 22 parts, among them J401 10103594-0001LF, J402 JST PH Battery Connector, Q401 P-Channel 1.25-W MOSFET, U401 3.3V_Reg, U403 LiPo Charger 500 mA, U404 1.8V_Reg

Commit message: Undocumented changes
Connections:
- wire segments 100 -> 99
Other:
- note added: "1) Charge battery while ON: V_BUS at 5V, battery connected, switch on.\n2) Charge battery while OFF: V_BUS at 5V, battery connected, switch off.\n3) Run on USB only: V_BUS at 5V, battery not connected, switch on.\n4) No long-term discharge allowed when batt present but off and not connected to USB."
- note added: "BATT"
- note added: "Datasheet for LP2985 suggests a Schottky to avoid\nreverse biasing Vin/Vout if that is a possibility but I don't expect that to happen."
- note added: "Main ON/OFF switch\nOn button board\nvia MCU board"
- note added: "V_BUS also comes\nfrom the UART header\nduring ICSP programming"
- note added: "What is leakage of V_BAT\nthrough mosfet and 100k resistor?"
- note removed: "1) Charge battery while running: V_BUS at 5V, battery connected, switch on.\n2) Charge battery while not running: V_BUS at 5V, battery connected, switch off.\n3) Run on USB only: V_BUS at 5V, battery not connected, switch on.\n4) No long-term discharge allowed when batt present but off and not connected to USB."
- note removed: "Datasheet suggests a Schottky to avoid reverse biasing Vin/Vout if that is a possibility but I don't expect that to happen."
- note removed: "These are connected \nat power switch on button board\nvia Arduino board"
- note removed: "V_BUS also comes\nfrom the UART header"
- note removed: "What is leakage of V_BAT through mosfet and 100k resistor?"
- note removed: "battery"
- moved on the sheet: C401, C404, C406, C407, C408, C410, J402, R404, U401, U404
