File: Boards/Flamingo PCBA/Flamingo PCB Rev 3/Flamingo PCB/Flamingo PCB.sch (KiCad schematic (older format))
At the start: 0 parts

Commit message: Undocumented changes
Changed lines of the file:
@@
 	2350 4050 3200 4050
 Wire Notes Line
-	3950 1550 3950 1350
+	3900 3550 3900 3350
 Wire Notes Line
-	4850 1350 4850 1550
-Text Notes 4150 1500 0    50   ~ 0
+	4800 3350 4800 3550
+Text Notes 4100 3500 0    50   ~ 0
 ICSP (pads)
 Wire Notes Line
-	3950 1350 4850 1350
+	3900 3350 4800 3350
 Wire Notes Line
-	4850 1550 3950 1550
-Text Notes 4150 1750 0    50   ~ 0
+	4800 3550 3900 3550
+Text Notes 4100 3750 0    50   ~ 0
 UART (header)
-Text Notes 4150 2000 0    50   ~ 0
+Text Notes 4100 4000 0    50   ~ 0
 Button Board
 Wire Notes Line
-	3950 1600 3950 1800
+	3900 3600 3900 3800
 Wire Notes Line
-	3950 1800 4850 1800
+	3900 3800 4800 3800
 Wire Notes Line
-	4850 1800 4850 1600
+	4800 3800 4800 3600
 Wire Notes Line
-	4850 1600 3950 1600
+	4800 3600 3900 3600
 Wire Notes Line
-	3950 2050 4850 2050
+	3900 4050 4800 4050
 Wire Notes Line
-	3950 2050 3950 1850
+	3900 4050 3900 3850
 Wire Notes Line
-	3950 1850 4850 1850
+	3900 3850 4800 3850
 Wire Notes Line
-	4850 1850 4850 2050
-Text Notes 4200 1300 0    39   ~ 0
+	4800 3850 4800 4050
+Text Notes 4150 3300 0    39   ~ 0
 Connectors
-Text Notes 1250 1950 0    50   ~ 0
+Text Notes 1250 3550 0    50   ~ 0
 Battery (JST-PH)
-Text Notes 1450 1750 0    39   ~ 0
+Text Notes 1450 3350 0    39   ~ 0
 Connectors
 Wire Notes Line
-	1150 2000 2050 2000
+	1150 3600 2050 3600
 Wire Notes Line
-	2050 2000 2050 1800
+	2050 3600 2050 3400
 Wire Notes Line
-	2050 1800 1150 1800
+	2050 3400 1150 3400
 Wire Notes Line
-	1150 1800 1150 2000
-Text Notes 4250 2250 0    50   ~ 0
+	1150 3400 1150 3600
+Text Notes 4200 4250 0    50   ~ 0
 APA102C
 Wire Notes Line
-	3950 2100 4850 2100
+	3900 4100 4800 4100
 Wire Notes Line
-	4850 2100 4850 2300
+	4800 4100 4800 4300
 Wire Notes Line
-	4850 2300 3950 2300
+	4800 4300 3900 4300
 Wire Notes Line
-	3950 2300 3950 2100
+	3900 4300 3900 4100
 $EndSCHEMATC
